File: 0101-SERIAL-CP2102N.kicad_sch (KiCad schematic)
At the start: 32 parts, among them J1 USB-C, J2 Conn_02x04_Odd_Even, Q1 DDC114TH, U1 CP2102N-A02-GQFN24

Commit message: Done PCB
Parts:
- removed D2, D3, D4, D5: LESD5Z5.0CT1G, Diode_SMD:D_SOD-523, symbol Diode:ESD9B5.0ST5G
- removed R6, R9: 0R, Resistor_SMD:R_0402_1005Metric, symbol Device:R_US
- added D10, D11, D8, D9: LESD5Z5.0CT1G, Diode_SMD:D_SOD-523, symbol Diode:ESD9B5.0ST5G
- R8: renamed from R7; footprint Resistor_SMD:R_0402_1005Metric -> Resistor_SMD:R_0603_1608Metric
- R9: renamed from R8; footprint Resistor_SMD:R_0402_1005Metric -> Resistor_SMD:R_0603_1608Metric
- renumbered D8 to D1, D9 to D2, D10 to D3, D11 to D4, D1 to D5, R10 to R12, R11 to R13, R12 to R14, R13 to R15
Connections:
- net CTS: now also J2.6 (Pin_6), D11.2 (A2); no longer J2.8 (Pin_8)
- net DTR: now also Q1.1 (E1), Q1.5 (B2)
- net DTR/RESET: now also J2.2 (Pin_2), D10.2 (A2); no longer J2.6 (Pin_6)
- net GND: now also J2.4 (Pin_4), D10.1 (A1), D11.1 (A1), D8.1 (A1), D9.1 (A1); no longer J2.1 (Pin_1)
- net RTS: now also Q1.2 (B1), Q1.4 (E2)
- net RTS/BOOT: now also J2.1 (Pin_1), D9.2 (A2); no longer D6.2 (A2), J2.4 (Pin_4)
- net RXD: now also J2.7 (Pin_7), D8.2 (A2); no longer D5.2 (A2), J2.3 (Pin_3)
- net TXD: now also D7.2 (A2), J2.8 (Pin_8); no longer J2.5 (Pin_5)
- net VBUS: now also D5.2 (A2), J2.3 (Pin_3); no longer D7.2 (A2), J2.2 (Pin_2)
- net VDD: now also D6.2 (A2), J2.5 (Pin_5); no longer J2.7 (Pin_7)
Other:
- moved on the sheet: D5

Commit message: Finish BOM
Parts:
- C1, C2: Manufacturer (none) -> SAMSUNG; PartNumber (none) -> C23733
- C3, C4: Manufacturer (none) -> SAMSUNG; PartNumber (none) -> C1525
- D1, D2: Manufacturer (none) -> EVERLIGHT; PartNumber (none) -> C72038
- Q1: value DDC114TH -> PUMH4,115; Manufacturer (none) -> Nexperia; PartNumber (none) -> C455002; Supplier (none) -> JLC-EXT
- R1: Manufacturer UniOhm -> YAGEO; PartNumber (none) -> C163478
- R2: Manufacturer UniOhm -> YAGEO; PartNumber (none) -> C137974
- R3: PartNumber (none) -> C11702
- U1: Manufacturer (none) -> SILICON LABS; PartNumber (none) -> C969151; Supplier (none) -> JLC-EXT
Other:
- note added: "Resistors of 10K are integrated in pin 2/5 of PUMH4,115"
- note removed: "Resistors of 10K are integrated in pin 2/5 of DDC114TH"
Changed lines of the file:
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@@
   (title_block
     (title "#0102 SERIAL-CP2102N")
-    (date "2022-09-29")
+    (date "2022-10-02")
     (rev "V1.0")
     (company "TileParts")
@@
     (stroke (width 0) (type default) (color 0 0 0 0))
   )
-  (text "Resistors of 10K are integrated\nin pin 2/5 of DDC114TH"
+  (text "Resistors of 10K are integrated\nin pin 2/5 of PUMH4,115"
     (at 127 83.82 0)
     (effects (font (size 1.27 1.27)) (justify left bottom))
@@
       (effects (font (size 1.27 1.27)) (justify right))
     )
-    (property "Value" "DDC114TH" (id 1) (at 147.32 62.23 90))
+    (property "Value" "PUMH4,115" (id 1) (at 147.32 62.23 90))
     (property "Footprint" "Package_TO_SOT_SMD:SOT-363_SC-70-6" (id 2) (at 149.86 60.96 0)
       (effects (font (size 1.27 1.27)) hide)
@@
       (effects (font (size 1.27 1.27)) hide)
     )
-    (property "Datasheet" "https://assets.nexperia.com/documents/data-sheet/PUMX1.pdf" (id 4) (at 147.32 55.88 0)
+    (property "Manufacturer" "Nexperia" (id 5) (at 147.32 55.88 0)
+      (effects (font (size 1.27 1.27)) hide)
+    )
+    (property "PartNumber" "C455002" (id 6) (at 147.32 55.88 0)
+      (effects (font (size 1.27 1.27)) hide)
+    )
+    (property "Supplier" "JLC-EXT" (id 7) (at 147.32 55.88 0)
       (effects (font (size 1.27 1.27)) hide)
     )
@@
       (effects (font (size 1.27 1.27)) hide)
     )
+    (property "PartNumber" "C11702" (id 6) (at 60.96 125.73 0)
+      (effects (font (size 1.27 1.27)) hide)
+    )
     (property "Supplier" "JLC" (id 5) (at 60.96 125.73 0)
       (effects (font (size 1.27 1.27)) hide)
@@
     )
     (property "Datasheet" "~" (id 3) (at 38.1 125.73 0)
+      (effects (font (size 1.27 1.27)) hide)
+    )
+    (property "Manufacturer" "SAMSUNG" (id 5) (at 38.1 125.73 0)
+      (effects (font (size 1.27 1.27)) hide)
+    )
+    (property "PartNumber" "C1525" (id 6) (at 38.1 125.73 0)
       (effects (font (size 1.27 1.27)) hide)
     )
@@
       (effects (font (size 1.27 1.27)) hide)
     )
-    (property "Manufacturer" "UniOhm" (id 4) (at 50.8 138.43 0)
+    (property "Manufacturer" "YAGEO" (id 4) (at 50.8 138.43 0)
+      (effects (font (size 1.27 1.27)) hide)
+    )
+    (property "PartNumber" "C163478" (id 6) (at 50.8 138.43 0)
       (effects (font (size 1.27 1.27)) hide)
     )
@@
     )
     (property "Datasheet" "https://www.silabs.com/documents/public/data-sheets/cp2102n-datasheet.pdf" (id 4) (at 73.66 152.4 0)
+      (effects (font (size 1.27 1.27)) hide)
+    )
+    (property "Manufacturer" "SILICON LABS" (id 5) (at 73.66 152.4 0)
+      (effects (font (size 1.27 1.27)) hide)
+    )
+    (property "PartNumber" "C969151" (id 6) (at 73.66 152.4 0)
+      (effects (font (size 1.27 1.27)) hide)
+    )
+    (property "Supplier" "JLC-EXT" (id 7) (at 73.66 152.4 0)
       (effects (font (size 1.27 1.27)) hide)
     )
@@
       (effects (font (size 1.27 1.27)) hide)
     )
+    (property "Manufacturer" "SAMSUNG" (id 5) (at 33.02 125.73 0)
+      (effects (font (size 1.27 1.27)) hide)
+    )
+    (property "PartNumber" "C23733" (id 6) (at 33.02 125.73 0)
+      (effects (font (size 1.27 1.27)) hide)
+    )
     (property "Supplier" "JLC" (id 4) (at 33.02 125.73 0)
       (effects (font (size 1.27 1.27)) hide)
@@
     )
     (property "Datasheet" "~" (id 3) (at 38.1 138.43 0)
+      (effects (font (size 1.27 1.27)) hide)
+    )
+    (property "Manufacturer" "SAMSUNG" (id 5) (at 38.1 138.43 0)
+      (effects (font (size 1.27 1.27)) hide)
+    )
+    (property "PartNumber" "C1525" (id 6) (at 38.1 138.43 0)
       (effects (font (size 1.27 1.27)) hide)
     )
@@
       (effects (font (size 1.27 1.27)) hide)
     )
+    (property "Manufacturer" "EVERLIGHT" (id 6) (at 240.03 44.45 0)
+      (effects (font (size 1.27 1.27)) hide)
+    )
+    (property "PartNumber" "C72038" (id 7) (at 240.03 44.45 0)
+      (effects (font (size 1.27 1.27)) hide)
+    )
     (property "Supplier" "JLC" (id 5) (at 240.03 44.45 0)
       (effects (font (size 1.27 1.27)) hide)
@@
     )
     (property "Datasheet" "~" (id 3) (at 240.03 49.53 0)
+      (effects (font (size 1.27 1.27)) hide)
+    )
+    (property "Manufacturer" "EVERLIGHT" (id 5) (at 240.03 49.53 0)
+      (effects (font (size 1.27 1.27)) hide)
+    )
+    (property "PartNumber" "C72038" (id 6) (at 240.03 49.53 0)
       (effects (font (size 1.27 1.27)) hide)
     )
@@
       (effects (font (size 1.27 1.27)) hide)
     )
+    (property "Manufacturer" "SAMSUNG" (id 6) (at 33.02 138.43 0)
+      (effects (font (size 1.27 1.27)) hide)
+    )
+    (property "PartNumber" "C23733" (id 7) (at 33.02 138.43 0)
+      (effects (font (size 1.27 1.27)) hide)
+    )
     (property "Supplier" "JLC" (id 5) (at 33.02 138.43 0)
       (effects (font (size 1.27 1.27)) hide)
@@
       (effects (font (size 1.27 1.27)) (justify right))
     )
-    (property "Value" "DDC114TH" (id 1) (at 147.32 64.77 90))
+    (property "Value" "PUMH4,115" (id 1) (at 147.32 64.77 90))
     (property "Footprint" "Package_TO_SOT_SMD:SOT-363_SC-70-6" (id 2) (at 144.78 66.04 0)
       (effects (font (size 1.27 1.27)) hide)
@@
     )
     (property "Datasheet" "https://assets.nexperia.com/documents/data-sheet/PUMX1.pdf" (id 4) (at 147.32 71.12 0)
+      (effects (font (size 1.27 1.27)) hide)
+    )
+    (property "Manufacturer" "Nexperia" (id 5) (at 147.32 71.12 0)
+      (effects (font (size 1.27 1.27)) hide)
+    )
+    (property "PartNumber" "C455002" (id 6) (at 147.32 71.12 0)
+      (effects (font (size 1.27 1.27)) hide)
+    )
+    (property "Supplier" "JLC-EXT" (id 7) (at 147.32 71.12 0)
       (effects (font (size 1.27 1.27)) hide)
     )
@@
       (effects (font (size 1.27 1.27)) hide)
     )
-    (property "Manufacturer" "UniOhm" (id 5) (at 50.8 146.05 0)
+    (property "Manufacturer" "YAGEO" (id 5) (at 50.8 146.05 0)
+      (effects (font (size 1.27 1.27)) hide)
+    )
+    (property "PartNumber" "C137974" (id 7) (at 50.8 146.05 0)
       (effects (font (size 1.27 1.27)) hide)
     )
@@
     )
     (path "/3df3307f-aca8-4c16-9be1-e03da0530051"
-      (reference "Q1") (unit 1) (value "DDC114TH") (footprint "Package_TO_SOT_SMD:SOT-363_SC-70-6")
+      (reference "Q1") (unit 1) (value "PUMH4,115") (footprint "Package_TO_SOT_SMD:SOT-363_SC-70-6")
     )
     (path "/f6b96ed6-751a-4520-a480-b81de293f8df"
-      (reference "Q1") (unit 2) (value "DDC114TH") (footprint "Package_TO_SOT_SMD:SOT-363_SC-70-6")
+      (reference "Q1") (unit 2) (value "PUMH4,115") (footprint "Package_TO_SOT_SMD:SOT-363_SC-70-6")
     )
     (path "/6d51830f-3c6c-4028-8d8c-030810e9a63c"

Commit message: Update MF docs V1.1
Parts:
- R1: Manufacturer YAGEO -> UniOhm; PartNumber C163478 -> C43473
- R2: Manufacturer YAGEO -> UniOhm; PartNumber C137974 -> C25896
- R8, R9: Manufacturer (none) -> UniOhm; PartNumber (none) -> C21189; Supplier (none) -> JLC
Changed lines of the file:
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@@
       (effects (font (size 1.27 1.27)) hide)
     )
-    (property "Manufacturer" "~" (id 4) (at 146.05 38.1 0)
-      (effects (font (size 1.27 1.27)) hide)
-    )
-    (property "PartNumber" "~" (id 5) (at 146.05 38.1 0)
-      (effects (font (size 1.27 1.27)) hide)
-    )
-    (property "Supplier" "~" (id 6) (at 146.05 38.1 0)
+    (property "Manufacturer" "UniOhm" (id 4) (at 146.05 38.1 0)
+      (effects (font (size 1.27 1.27)) hide)
+    )
+    (property "PartNumber" "C21189" (id 5) (at 146.05 38.1 0)
+      (effects (font (size 1.27 1.27)) hide)
+    )
+    (property "Supplier" "JLC" (id 6) (at 146.05 38.1 0)
       (effects (font (size 1.27 1.27)) hide)
     )
@@
       (effects (font (size 1.27 1.27)) hide)
     )
-    (property "Manufacturer" "~" (id 4) (at 146.05 43.18 0)
-      (effects (font (size 1.27 1.27)) hide)
-    )
-    (property "PartNumber" "~" (id 5) (at 146.05 43.18 0)
-      (effects (font (size 1.27 1.27)) hide)
-    )
-    (property "Supplier" "~" (id 6) (at 146.05 43.18 0)
+    (property "Manufacturer" "UniOhm" (id 4) (at 146.05 43.18 0)
+      (effects (font (size 1.27 1.27)) hide)
+    )
+    (property "PartNumber" "C21189" (id 5) (at 146.05 43.18 0)
+      (effects (font (size 1.27 1.27)) hide)
+    )
+    (property "Supplier" "JLC" (id 6) (at 146.05 43.18 0)
       (effects (font (size 1.27 1.27)) hide)
     )
@@
       (effects (font (size 1.27 1.27)) hide)
     )
-    (property "Manufacturer" "YAGEO" (id 4) (at 50.8 138.43 0)
-      (effects (font (size 1.27 1.27)) hide)
-    )
-    (property "PartNumber" "C163478" (id 6) (at 50.8 138.43 0)
+    (property "Manufacturer" "UniOhm" (id 4) (at 50.8 138.43 0)
+      (effects (font (size 1.27 1.27)) hide)
+    )
+    (property "PartNumber" "C43473" (id 6) (at 50.8 138.43 0)
       (effects (font (size 1.27 1.27)) hide)
     )
@@
       (effects (font (size 1.27 1.27)) hide)
     )
-    (property "Manufacturer" "YAGEO" (id 5) (at 50.8 146.05 0)
-      (effects (font (size 1.27 1.27)) hide)
-    )
-    (property "PartNumber" "C137974" (id 7) (at 50.8 146.05 0)
-      (effects (font (size 1.27 1.27)) hide)
-    )
+    (property "Manufacturer" "UniOhm" (id 5) (at 50.8 146.05 0)
+      (effects (font (size 1.27 1.27)) hide)
+    )
+    (property "PartNumber" "C25896" (id 7) (at 50.8 146.05 0)
+      (effects (font (size 1.27 1.27)) hide)
+    )
